File: kicad/io-master-dev-board.kicad_pcb (KiCad board)
At the start: 4 copper layers, 170 x 100 mm, 674 parts, among them J1 54-00166, J2 10118193, J3 0.1" HDR, J4 0.1" HDR, Q1 Q_NPN_BCE, Q10 DMN63D8LDW, Q11 DMN63D8LDW, Q12 MMBT3906, Q13 DMN63D8LDW, Q14 MMBT3906, Q15 DMN63D8LDW, Q16 MMBT3906, Q17 MMBT3904, Q18 MMBT3906, Q19 DMG1029SV, Q2 Q_NPN_BCE, Q20 MMBT3904, Q21 MMBT3906, Q22 DMG1029SV, Q23 MMBT3904, Q24 DMN63D8LDW, Q25 DMN63D8LDW, Q26 MMBT3906, Q27 DMP3099L, Q3 MMBT3904, Q4 MMBT3906, Q5 DMG1029SV, Q6 MMBT3904, Q7 MMBT3906, Q8 DMG1029SV, Q9 MMBT3904, SW1 JS202011SCQN, SW2 EVQ-Q2B03W, U1 AZ1117-3.3, U10 PI5A3157, U11 LM7171, U12 LM7171, U13 LM7171, U14 DG449, U15 LM7171, U16 LM7171, U17 DG448DV, U18 DG448DV, U19 NCV20074, U2 STM32H743ZITx, U20 NCV20074, U21 NCV20074, U22 MCP4728A2, U23 NCV20074, U24 TS3011, U25 MCP4725A1, U26 TS3011, U27 PI5A3157, U28 LM7171, U29 LM7171, U3 USB3300-EZK, U30 LM7171, U31 DG449, U32 LM7171, U33 LM7171, U34 DG448DV, U35 DG448DV, U36 ADP5070AREZ, U37 NCV20074, U4 LM2621, U5 MCP4728A0, U6 NCV20074, U7 TS3011, U8 MCP4725A0, U9 TS3011, Y1 48MHz, Y2 24MHz

Commit message: WIP board layout
Parts:
- removed C100, C41, C46, C64, C65, C66, C67, C90, C91, C92, C93: 10u, Capacitor_SMD:C_0805_2012Metric
- removed C101, C106, C43: 1u, Capacitor_SMD:C_0603_1608Metric
- removed C102, C103, C55, C56, C59, C81, C82, C85: C, Capacitor_SMD:C_0603_1608Metric
- removed C104: 0.22u, Capacitor_SMD:C_0603_1608Metric
- removed C105: 82p, Capacitor_SMD:C_0603_1608Metric
- removed C107, C108: 22u, Capacitor_SMD:C_1210_3225Metric
- removed C109, C110, C40, C45, C99: C, Capacitor_SMD:C_1210_3225Metric
- removed C111, C112, C113, C114, C115, C116, C117, C118, C36, C38, C39, C42, C47, C48, C49, C50, C51, C52, C53, C54, C57, C58, C60, C61, C62, C63, C68, C69, C70, C71, C73, C74, C75, C76, C77, C78, C79, C80, C83, C84, C86, C87, C88, C89, C94, C95, C96, C97: 0.1u, Capacitor_SMD:C_0603_1608Metric
- removed C37: 4.7u, Capacitor_SMD:C_0805_2012Metric
- removed C44: 33p, Capacitor_SMD:C_0603_1608Metric
- removed C72, C98: 1000p, Capacitor_SMD:C_0603_1608Metric
- removed D10: RGB, io-master:LED_Everlight_19-337C
- removed D11, D7, D8, D9: YEL/GRN, io-master:LED_Kingbright_APTB1615YSGC
- removed D12: DDZ5V6ASF, Diode_SMD:D_SOD-323F
- removed D13, D30, D31: NSR0530HT1G, Diode_SMD:D_SOD-323
- removed D14, D15, D28, D29: MM3Z9V1ST1G, Diode_SMD:D_SOD-323
- removed D16, D20, D24, D32, D36, D37, D38, D39: MM3Z15VST1G, Diode_SMD:D_SOD-323
- removed D17, D18, D21, D22, D25, D26, D33, D34: 1N4148, Diode_SMD:D_SOD-323
- removed D19, D23, D27, D35: RED, LED_SMD:LED_0603_1608Metric
- removed D4, D5: BLUE, LED_SMD:LED_0603_1608Metric
- removed D6: GREEN, LED_SMD:LED_0603_1608Metric
- removed F1: 0.5A, Fuse:Fuse_1206_3216Metric
- removed F2: 0.1A, Fuse:Fuse_1206_3216Metric
- removed L1: 82u, io-master:L_Bourns_SRF0703
- removed L2: 10u, io-master:L_Abracon_ASPI-0418FS
- removed L3: 15u, Inductor_SMD:L_Taiyo-Yuden_NR-50xx
- removed Q1, Q2: Q_NPN_BCE, Package_TO_SOT_SMD:SOT-323_SC-70
- removed Q10, Q11, Q13, Q15, Q24, Q25: DMN63D8LDW, Package_TO_SOT_SMD:SOT-363_SC-70-6
- removed Q12, Q14, Q16, Q18, Q21, Q26, Q4, Q7: MMBT3906, Package_TO_SOT_SMD:SOT-323_SC-70
- removed Q17, Q20, Q23, Q3, Q6, Q9: MMBT3904, Package_TO_SOT_SMD:SOT-323_SC-70
- removed Q19, Q22, Q5, Q8: DMG1029SV, Package_TO_SOT_SMD:SOT-563
- removed Q27: DMP3099L, Package_TO_SOT_SMD:SOT-23
- removed R100, R101, R108, R109, R116, R124, R125, R136, R137, R139, R140, R151, R152, R154, R155, R166, R167, R212, R213, R216, R217, R218, R219, R226, R227, R234, R248, R249, R260, R261, R43, R49, R94, R95, R98, R99: 10K, Resistor_SMD:R_0603_1608Metric
- removed R102, R103, R104, R105, R106, R107, R112, R113, R117, R118, R126, R127, R128, R129, R130, R131, R132, R133, R135, R14, R141, R142, R143, R144, R145, R146, R147, R148, R15, R150, R156, R157, R158, R159, R160, R161, R162, R163, R165, R168, R169, R17, R170, R171, R172, R173, R174, R175, R192, R193, R20, R201, R206, R207, R21, R214, R215, R220, R221, R222, R223, R224, R225, R23, R230, R231, R235, R236, R24, R25, R250, R251, R252, R253, R254, R255, R256, R257, R259, R26, R262, R31, R32, R34, R35, R36, R37, R38, R41, R42, R50, R51, R52, R53, R54, R55, R56, R57, R74, R75, R83, R88, R89, R96, R97: 100K, Resistor_SMD:R_0603_1608Metric
- removed R110, R111, R114, R115, R228, R229, R232, R233: 0, Resistor_SMD:R_0603_1608Metric
- removed R119, R120, R121, R122, R237, R238, R239, R240: 120, Resistor_SMD:R_0805_2012Metric
- removed R123, R138, R153, R247: 2, Resistor_SMD:R_0603_1608Metric
- removed R13, R19, R22, R30, R33, R39, R40: 1K, Resistor_SMD:R_0603_1608Metric
- removed R134, R149, R164, R258: 6.8K, Resistor_SMD:R_0603_1608Metric
- removed R16, R18: 4.7K, Resistor_SMD:R_0603_1608Metric
- removed R176, R177, R178, R179, R180, R181, R182, R183, R194, R198, R200, R203, R48, R58, R59, R60, R61, R62, R63, R64, R65, R76, R80, R82, R85: 110K, Resistor_SMD:R_0603_1608Metric
- removed R184, R185, R186, R187, R188, R189, R190, R191, R197, R199, R202, R205, R46, R66, R67, R68, R69, R70, R71, R72, R73, R79, R81, R84, R87: 1M, Resistor_SMD:R_0603_1608Metric
- removed R195, R196, R209, R77, R78, R91: R, Resistor_SMD:R_0603_1608Metric
- removed R204, R208, R210, R211, R86, R90, R92, R93: 47K, Resistor_SMD:R_0603_1608Metric
- removed R241: 5.36K, Resistor_SMD:R_0603_1608Metric
- removed R242: 390K, Resistor_SMD:R_0603_1608Metric
- removed R243: 2.43M, Resistor_SMD:R_0603_1608Metric
- removed R244: 137K, Resistor_SMD:R_0603_1608Metric
- removed R245: 118K, Resistor_SMD:R_0603_1608Metric
- removed R246: 2.32M, Resistor_SMD:R_0603_1608Metric
- removed R27, R28, R29: 330, Resistor_SMD:R_0603_1608Metric
- removed R44: 820, Resistor_SMD:R_0603_1608Metric
- removed R45: 12K, Resistor_SMD:R_0603_1608Metric
- removed R47: 220K, Resistor_SMD:R_0603_1608Metric
- removed REF**: Symbol_Barrel_Polarity, Symbol:Symbol_Barrel_Polarity
- removed REF**: OSHW-Logo_5.7x6mm_Copper, Symbol:OSHW-Logo_5.7x6mm_Copper
- removed REF**: OSHW-Logo_5.7x6mm_Mask, io-master:OSHW-Logo_5.7x6mm_Mask
- removed TP10, TP109, TP11, TP12, TP120, TP121, TP125, TP126, TP127, TP128, TP129, TP13, TP130, TP131, TP132, TP133, TP134, TP135, TP136, TP137, TP138, TP139, TP14, TP140, TP149, TP15, TP150, TP154, TP155, TP156, TP157, TP158, TP159, TP160, TP171, TP172, TP173, TP5, TP6, TP7, TP8, TP9: TestPoint, TestPoint:TestPoint_Pad_D1.0mm
- removed TP100: TRIS8, TestPoint:TestPoint_Pad_D1.0mm
- removed TP101: SCL, TestPoint:TestPoint_Pad_D1.0mm
- removed TP102: SDA, TestPoint:TestPoint_Pad_D1.0mm
- removed TP103: VSET, TestPoint:TestPoint_Pad_D1.0mm
- removed TP104: PD1, TestPoint:TestPoint_Pad_D1.0mm
- removed TP105: PD2, TestPoint:TestPoint_Pad_D1.0mm
- removed TP106: PD3, TestPoint:TestPoint_Pad_D1.0mm
- removed TP107: PD4, TestPoint:TestPoint_Pad_D1.0mm
- removed TP108: SW, TestPoint:TestPoint_Pad_D1.0mm
- removed TP110: FB, TestPoint:TestPoint_Pad_D1.0mm
- removed TP111: Vout, TestPoint:TestPoint_Pad_D1.0mm
- removed TP112: DVH1, TestPoint:TestPoint_Pad_D1.0mm
- removed TP113: DVL1, TestPoint:TestPoint_Pad_D1.0mm
- removed TP114: DVH2, TestPoint:TestPoint_Pad_D1.0mm
- removed TP115: DVL2, TestPoint:TestPoint_Pad_D1.0mm
- removed TP116: VH1, TestPoint:TestPoint_Pad_D1.0mm
- removed TP117: VL1, TestPoint:TestPoint_Pad_D1.0mm
- removed TP118: VH2, TestPoint:TestPoint_Pad_D1.0mm
- removed TP119: VL2, TestPoint:TestPoint_Pad_D1.0mm
- removed TP122: TH12, TestPoint:TestPoint_Pad_D1.0mm
- removed TP123: 1-2, TestPoint:TestPoint_Pad_D1.0mm
- removed TP124: TH1, TestPoint:TestPoint_Pad_D1.0mm
- removed TP141: DVH3, TestPoint:TestPoint_Pad_D1.0mm
- removed TP142: DVL3, TestPoint:TestPoint_Pad_D1.0mm
- removed TP143: DVH4, TestPoint:TestPoint_Pad_D1.0mm
- removed TP144: DVL4, TestPoint:TestPoint_Pad_D1.0mm
- removed TP145: VH3, TestPoint:TestPoint_Pad_D1.0mm
- removed TP146: VL3, TestPoint:TestPoint_Pad_D1.0mm
- removed TP147: VH4, TestPoint:TestPoint_Pad_D1.0mm
- removed TP148: VL4, TestPoint:TestPoint_Pad_D1.0mm
- removed TP151: TH34, TestPoint:TestPoint_Pad_D1.0mm
- removed TP152: 3-4, TestPoint:TestPoint_Pad_D1.0mm
- removed TP153: TH3, TestPoint:TestPoint_Pad_D1.0mm
- removed TP16: VIN, TestPoint:TestPoint_Pad_D1.0mm
- removed TP161: SS, TestPoint:TestPoint_Pad_D1.0mm
- removed TP162: SLEW, TestPoint:TestPoint_Pad_D1.0mm
- removed TP163: SEQ, TestPoint:TestPoint_Pad_D1.0mm
- removed TP164: INBK, TestPoint:TestPoint_Pad_D1.0mm
- removed TP165: SW2, TestPoint:TestPoint_Pad_D1.0mm
- removed TP166: SW1, TestPoint:TestPoint_Pad_D1.0mm
- removed TP167: FB1, TestPoint:TestPoint_Pad_D1.0mm
- removed TP168: FB2, TestPoint:TestPoint_Pad_D1.0mm
- removed TP169: +15V, TestPoint:TestPoint_Pad_D1.0mm
- removed TP17: DCIN, TestPoint:TestPoint_Pad_D1.0mm
- removed TP170: -15V, TestPoint:TestPoint_Pad_D1.0mm
- removed TP174: PRST, TestPoint:TestPoint_Pad_D1.0mm
- removed TP18: VBUS, TestPoint:TestPoint_Pad_D1.0mm
- removed TP19: 3.3V, TestPoint:TestPoint_Pad_D1.0mm
- removed TP20: PU5, TestPoint:TestPoint_Pad_D1.0mm
- removed TP21: PD5, TestPoint:TestPoint_Pad_D1.0mm
- removed TP22: PU6, TestPoint:TestPoint_Pad_D1.0mm
- removed TP23: PD6, TestPoint:TestPoint_Pad_D1.0mm
- removed TP24: PU7, TestPoint:TestPoint_Pad_D1.0mm
- removed TP25: PD7, TestPoint:TestPoint_Pad_D1.0mm
- removed TP26: PU8, TestPoint:TestPoint_Pad_D1.0mm
- removed TP27: PD8, TestPoint:TestPoint_Pad_D1.0mm
- removed TP28: PG8, TestPoint:TestPoint_Pad_D1.0mm
- removed TP29: PG9, TestPoint:TestPoint_Pad_D1.0mm
- removed TP30: PG10, TestPoint:TestPoint_Pad_D1.0mm
- removed TP31: PG11, TestPoint:TestPoint_Pad_D1.0mm
- removed TP32: PG12, TestPoint:TestPoint_Pad_D1.0mm
- removed TP33: PG13, TestPoint:TestPoint_Pad_D1.0mm
- removed TP34: PG14, TestPoint:TestPoint_Pad_D1.0mm
- removed TP35: PG15, TestPoint:TestPoint_Pad_D1.0mm
- removed TP36: PF3, TestPoint:TestPoint_Pad_D1.0mm
- removed TP37: PF4, TestPoint:TestPoint_Pad_D1.0mm
- removed TP38: PF5, TestPoint:TestPoint_Pad_D1.0mm
- removed TP39: PF6, TestPoint:TestPoint_Pad_D1.0mm
- removed TP4: GND, TestPoint:TestPoint_Keystone_5010-5014_Multipurpose
- removed TP40: PF7, TestPoint:TestPoint_Pad_D1.0mm
- removed TP41: PF8, TestPoint:TestPoint_Pad_D1.0mm
- removed TP42: PF9, TestPoint:TestPoint_Pad_D1.0mm
- removed TP43: PF10, TestPoint:TestPoint_Pad_D1.0mm
- removed TP44: PF11, TestPoint:TestPoint_Pad_D1.0mm
- removed TP45: PF12, TestPoint:TestPoint_Pad_D1.0mm
- removed TP46: PF13, TestPoint:TestPoint_Pad_D1.0mm
- removed TP47: PF14, TestPoint:TestPoint_Pad_D1.0mm
- removed TP48: PF15, TestPoint:TestPoint_Pad_D1.0mm
- removed TP49: PE0, TestPoint:TestPoint_Pad_D1.0mm
- removed TP50: PE1, TestPoint:TestPoint_Pad_D1.0mm
- removed TP51: PE2, TestPoint:TestPoint_Pad_D1.0mm
- removed TP52: PE3, TestPoint:TestPoint_Pad_D1.0mm
- removed TP53: PE4, TestPoint:TestPoint_Pad_D1.0mm
- removed TP54: PE5, TestPoint:TestPoint_Pad_D1.0mm
- removed TP55: PE6, TestPoint:TestPoint_Pad_D1.0mm
- removed TP56: PE7, TestPoint:TestPoint_Pad_D1.0mm
- removed TP57: PE12, TestPoint:TestPoint_Pad_D1.0mm
- removed TP58: PE13, TestPoint:TestPoint_Pad_D1.0mm
- removed TP59: PE14, TestPoint:TestPoint_Pad_D1.0mm
- removed TP60: PE15, TestPoint:TestPoint_Pad_D1.0mm
- removed TP61: OUT1, TestPoint:TestPoint_Pad_D1.0mm
- removed TP62: OUT2, TestPoint:TestPoint_Pad_D1.0mm
- removed TP63: OUT3, TestPoint:TestPoint_Pad_D1.0mm
- removed TP64: OUT4, TestPoint:TestPoint_Pad_D1.0mm
- removed TP65: IN1, TestPoint:TestPoint_Pad_D1.0mm
- removed TP66: IN2, TestPoint:TestPoint_Pad_D1.0mm
- removed TP67: IN3, TestPoint:TestPoint_Pad_D1.0mm
- removed TP68: IN4, TestPoint:TestPoint_Pad_D1.0mm
- removed TP69: TRIS1, TestPoint:TestPoint_Pad_D1.0mm
- removed TP70: TRIS2, TestPoint:TestPoint_Pad_D1.0mm
- removed TP71: TRIS3, TestPoint:TestPoint_Pad_D1.0mm
- removed TP72: TRIS4, TestPoint:TestPoint_Pad_D1.0mm
- removed TP73: DIFF12, TestPoint:TestPoint_Pad_D1.0mm
- removed TP74: TERM12, TestPoint:TestPoint_Pad_D1.0mm
- removed TP75: DIFF34, TestPoint:TestPoint_Pad_D1.0mm
- removed TP76: TERM34, TestPoint:TestPoint_Pad_D1.0mm
- removed TP77: PU1, TestPoint:TestPoint_Pad_D1.0mm
- removed TP78: PU2, TestPoint:TestPoint_Pad_D1.0mm
- removed TP79: PU3, TestPoint:TestPoint_Pad_D1.0mm
- removed TP80: PU4, TestPoint:TestPoint_Pad_D1.0mm
- removed TP82: TXO, TestPoint:TestPoint_Pad_D1.0mm
- removed TP83: RXI, TestPoint:TestPoint_Pad_D1.0mm
- removed TP84: DM, TestPoint:TestPoint_Pad_D1.0mm
- removed TP85: DP, TestPoint:TestPoint_Pad_D1.0mm
- removed TP89: DIFF78, TestPoint:TestPoint_Pad_D1.0mm
- removed TP90: TERM78, TestPoint:TestPoint_Pad_D1.0mm
- removed TP91: DIFF56, TestPoint:TestPoint_Pad_D1.0mm
- removed TP92: TERM56, TestPoint:TestPoint_Pad_D1.0mm
- removed TP93: OUT5, TestPoint:TestPoint_Pad_D1.0mm
- removed TP94: OUT6, TestPoint:TestPoint_Pad_D1.0mm
- removed TP95: OUT7, TestPoint:TestPoint_Pad_D1.0mm
- removed TP96: OUT8, TestPoint:TestPoint_Pad_D1.0mm
- removed TP97: TRIS5, TestPoint:TestPoint_Pad_D1.0mm
- removed TP98: TRIS6, TestPoint:TestPoint_Pad_D1.0mm
- removed TP99: TRIS7, TestPoint:TestPoint_Pad_D1.0mm
- removed U10, U27: PI5A3157, Package_TO_SOT_SMD:SOT-363_SC-70-6
- removed U11, U12, U13, U15, U16, U28, U29, U30, U32, U33: LM7171, Package_SO:SOIC-8_3.9x4.9mm_P1.27mm
- removed U14, U31: DG449, Package_TO_SOT_SMD:SOT-23-8
- removed U17, U18, U34, U35: DG448DV, Package_SO:TSOP-6_1.65x3.05mm_P0.95mm
- removed U19, U20, U21, U23, U37, U6: NCV20074, Package_SO:TSSOP-14_4.4x5mm_P0.65mm
- removed U22: MCP4728A2, Package_SO:MSOP-10_3x3mm_P0.5mm
- removed U24, U26, U7, U9: TS3011, Package_TO_SOT_SMD:SOT-353_SC-70-5
- removed U25: MCP4725A1, Package_TO_SOT_SMD:SOT-23-6
- removed U36: ADP5070AREZ, Package_SO:ETSSOP-20-1EP_4.4x6.5mm_P0.65mm_EP3x4.2mm
- removed U5: MCP4728A0, Package_SO:MSOP-10_3x3mm_P0.5mm
- removed U8: MCP4725A0, Package_TO_SOT_SMD:SOT-23-6
- added J10: Conn_01x27, Connector_PinHeader_1.27mm:PinHeader_1x27_P1.27mm_Vertical, F.Cu at (104.3, 53.8)
- added J11: 0.1" HDR, Connector_PinSocket_2.54mm:PinSocket_2x05_P2.54mm_Vertical, F.Cu at (90.0, 110.0)
- added J5: UART, Connector_PinHeader_2.54mm:PinHeader_1x06_P2.54mm_Horizontal, F.Cu at (36.5, 106.5)
- added J6: Conn_02x32_Odd_Even, Connector_PinHeader_1.27mm:PinHeader_2x32_P1.27mm_Vertical, F.Cu at (98.0, 89.4)
- added J7: Conn_02x27_Odd_Even, Connector_PinHeader_1.27mm:PinHeader_2x27_P1.27mm_Vertical, F.Cu at (98.0, 53.8)
- added J8: Conn_01x10, Connector_PinHeader_1.27mm:PinHeader_1x10_P1.27mm_Vertical, F.Cu at (104.3, 39.8)
- added J9: Conn_01x32, Connector_PinHeader_1.27mm:PinHeader_1x32_P1.27mm_Vertical, F.Cu at (104.3, 89.4)
- added JP1: Jumper_NO_Small, Resistor_SMD:R_0603_1608Metric, F.Cu at (44.5, 50.5)
- added JP2: Jumper_NC_Small, Resistor_SMD:R_0603_1608Metric, F.Cu at (43.0, 50.5)
- C1: value 0.47u -> 0.1u
- C10: value 1u -> 0.1u
- C11: value 1u -> 20p
- C13: value 20p -> 10u; footprint Capacitor_SMD:C_0603_1608Metric -> Capacitor_SMD:C_0805_2012Metric
- C14: value 2.2u -> 22u; footprint Capacitor_SMD:C_0805_2012Metric -> Capacitor_SMD:C_1210_3225Metric
- C16, C9: value 0.1u -> 4.7u; footprint Capacitor_SMD:C_0603_1608Metric -> Capacitor_SMD:C_0805_2012Metric
- C18, C19: value 0.1u -> 1u
- C2: value 1u -> 4.7u; footprint Capacitor_SMD:C_0603_1608Metric -> Capacitor_SMD:C_0805_2012Metric
- C20, C24: value 0.1u -> 2.2u; footprint Capacitor_SMD:C_0603_1608Metric -> Capacitor_SMD:C_0805_2012Metric
- C29, C8: value 4.7u -> 0.1u; footprint Capacitor_SMD:C_0805_2012Metric -> Capacitor_SMD:C_0603_1608Metric
- C4: value 10u -> 0.1u; footprint Capacitor_SMD:C_0805_2012Metric -> Capacitor_SMD:C_0603_1608Metric
- C5: value 22u -> 0.1u; footprint Capacitor_SMD:C_1210_3225Metric -> Capacitor_SMD:C_0603_1608Metric
- C7: value 2.2u -> 0.1u; footprint Capacitor_SMD:C_0805_2012Metric -> Capacitor_SMD:C_0603_1608Metric
- D1: value B130L -> DDZ5V6ASF; footprint Diode_SMD:D_SMA -> Diode_SMD:D_SOD-323F
- D2: value B130L -> ORANGE; footprint Diode_SMD:D_SMA -> LED_SMD:LED_0603_1608Metric
- D3: value ORANGE -> RGB; footprint LED_SMD:LED_0603_1608Metric -> io-master-dev-board:LED_Everlight_19-337C
- J1: value 54-00166 -> USB4110-GF-A; footprint io-master:BarrelJack_Tensility_54-00166_Horizontal -> io-master-dev-board:USB_C_Receptable_GCT_USB4110
- J2: value 10118193 -> Conn_01x08; footprint io-master:USB_Micro-B_Amphenol_10118193-0001LF_Horizontal -> Connector_PinHeader_2.54mm:PinHeader_1x08_P2.54mm_Vertical
- J3: value 0.1" HDR -> Conn_01x08; footprint io-master:PinSocket_2x05_P2.54mm_Vertical_AltNumbering -> Connector_PinHeader_2.54mm:PinHeader_1x08_P2.54mm_Vertical
- J4: value 0.1" HDR -> Conn_01x12; footprint Connector_PinSocket_2.54mm:PinSocket_2x05_P2.54mm_Vertical -> Connector_PinHeader_2.54mm:PinHeader_1x12_P2.54mm_Vertical
- R1: value R -> 900K
- R10, R12: value 100K -> 330
- R11: value 1K -> 330
- R2: value R -> 820
- R3: value R -> 1M
- R4: value R -> 10K
- R5: value 1K -> 12K
- R6: value 10K -> 1K
- R9: value R -> 4.7K
- SW1: footprint io-master:SW_DPDT_CK_JS202011SCQN -> io-master-dev-board:SW_DPDT_CK_JS202011SCQN
- SW2: value EVQ-Q2B03W -> 222LMVAAR; footprint Button_Switch_SMD:SW_SPST_EVQQ2 -> io-master-dev-board:SW_Push_CTS_222LMVA
- TP1, TP3: value TestPoint -> GND; footprint TestPoint:TestPoint_Pad_D1.0mm -> TestPoint:TestPoint_Keystone_5010-5014_Multipurpose
- TP2: value TestPoint -> VBUS
- U1: value AZ1117-3.3 -> TUSB320; footprint Package_TO_SOT_SMD:SOT-223-3_TabPin2 -> Package_DFN_QFN:Texas_X2QFN-12_1.6x1.6mm_P0.4mm
- U2: value STM32H743ZITx -> K7803JT-500R3; footprint Package_QFP:LQFP-144_20x20mm_P0.5mm -> io-master-dev-board:DCDC_Module_K78xxJT-500R3
- U4: value LM2621 -> STM32H743ZITx; footprint Package_SO:VSSOP-8_3.0x3.0mm_P0.65mm -> Package_QFP:LQFP-144_20x20mm_P0.5mm
- Y1: value 48MHz -> 24MHz; footprint io-master:Crystal_SMD_Murata_XRCGB -> io-master-dev-board:Crystal_SMD_Murata_XRCGB
- Y2: value 24MHz -> 48MHz; footprint io-master:Crystal_SMD_Murata_XRCGB -> io-master-dev-board:Crystal_SMD_Murata_XRCGB
- moved C18 158.9 mm to (-4.50, 148.0)
- moved R1 128.0 mm to (42.5, 47.5), turned to 180 degrees
- moved J3 127.4 mm to (72.0, 36.5), turned to 270 degrees
- moved TP1 123.5 mm to (44.5, 36.5)
- moved R2 120.8 mm to (50.5, 57.0), turned to 180 degrees
- moved TP3 106.3 mm to (99.0, 113.5)
- moved R11 103.3 mm to (1.00, 142.0)
- moved R12 101.4 mm to (-14.0, 100.0)
- moved H4 95.5 mm to (100.0, 135.0)
- moved H2 95.0 mm to (100.0, 35.0)
- moved C14 93.9 mm to (-12.5, 104.0)
- moved C23 92.7 mm to (-12.5, 95.5)
- moved R4 89.9 mm to (45.5, 47.5), turned to 180 degrees
- moved R10 87.3 mm to (0.00, 91.5)
- moved C24 87.3 mm to (-7.00, 107.5)
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Connections:
- C1 pad 1: GND -> +3V3
- C1 pad 2: CHASSIS -> GND
- C10 pad 1: /3.3V -> /VDDA1.8
- C11 pad 1: /3.3V -> Net-(C11-Pad1)
- C12 pad 1: /Microcontroller/OSC_OUT -> Net-(C12-Pad1)
- C13 pad 1: /Microcontroller/OSC_IN -> VBUS
- C14 pad 1: /Microcontroller/VCAP -> +3V3
- C15 pad 1: /3.3V -> +3V3
- C16 pad 1: /3.3V -> +3V3
- C17 pad 1: /3.3V -> +3V3
- C18 pad 1: GND -> +3V3
- C18 pad 2: /-15V -> GND
- C19 pad 1: /3.3V -> +3V3
- C2 pad 1: /Microcontroller/USB_VBUS -> /VDD1.8
- C20 pad 1: /3.3V -> /Microcontroller/VCAP
- C21 pad 1: GND -> +3V3
- C21 pad 2: /-15V -> GND
- C22 pad 1: /3.3V -> +3V3
- C23 pad 1: /3.3V -> +3V3
- C24 pad 1: /3.3V -> /Microcontroller/VCAP
- C25 pad 1: /3.3V -> +3V3
- C26 pad 1: /3.3V -> +3V3
- C27 pad 1: /3.3V -> +3V3
- C28 pad 1: Net-(C28-Pad1) -> +3V3
- C29 pad 1: /Microcontroller/VDD1.8 -> +3V3
- C3 pad 1: /Vin -> +3V3
- C30 pad 1: /Microcontroller/VDD1.8 -> +3V3
- C31 pad 1: /3.3V -> +3V3
- C32 pad 1: /Microcontroller/VDD1.8 -> +3V3
- C33 pad 1: /Microcontroller/XO -> Net-(C33-Pad1)
- C34 pad 1: /Microcontroller/XI -> Net-(C34-Pad1)
- C35 pad 1: /3.3V -> /Microcontroller/~RESET
- C4 pad 1: /Vin -> /VDD1.8
- C5 pad 1: /3.3V -> /VDD1.8
- C6 pad 1: /3.3V -> +3V3
- C7 pad 1: /Microcontroller/VCAP -> GND
- C7 pad 2: GND -> Net-(C7-Pad2)
- C8 pad 1: /3.3V -> +3V3
- C9 pad 1: /3.3V -> /VDDA1.8
- D1 pad 2: Net-(D1-Pad2) -> GND
- D2 pad 1: Net-(D1-Pad1) -> Net-(D2-Pad1)
- D2 pad 2: Net-(D2-Pad2) -> +3V3
- D3 pad 1: Net-(D3-Pad1) -> GND
- D3 pad 2: /3.3V -> Net-(D3-Pad2)
- FB1 pad 1: /3.3V -> +3V3
- H1 pad 1: CHASSIS -> GND
- H2 pad 1: CHASSIS -> GND
- H3 pad 1: CHASSIS -> GND
- H4 pad 1: CHASSIS -> GND
- J2 pad 1: /Microcontroller/USB_VBUS -> /Microcontroller/PG8
- J2 pad 2: /D- -> /Microcontroller/PG9
- J2 pad 3: /D+ -> /Microcontroller/PG10
- J2 pad 4: Net-(J2-Pad4) -> /Microcontroller/PG11
- J2 pad 5: GND -> /Microcontroller/PG12
- J2 pad 6: CHASSIS -> /Microcontroller/PG13
- J3 pad 1: /Circuit Protection - I/O Pin 1/TARGET_IO_1 -> /Microcontroller/PE0
- J3 pad 2: /Circuit Protection - I/O Pin 2/TARGET_IO_2 -> /Microcontroller/PE1
- J3 pad 3: /Circuit Protection - I/O Pin 3/TARGET_IO_3 -> /Microcontroller/PE2
- J3 pad 4: /Circuit Protection - I/O Pin 4/TARGET_IO_4 -> /Microcontroller/PE3
- J3 pad 5: Net-(F2-Pad2) -> /Microcontroller/PE4
- J3 pad 6: GND -> /Microcontroller/PE5
- J3 pad 7: GND -> /Microcontroller/PE6
- J3 pad 8: GND -> /Microcontroller/PE7
- J4 pad 1: /3.3V -> /Microcontroller/PF4
- J4 pad 10: /Microcontroller/nRESET -> /Microcontroller/PF13
- J4 pad 2: /Microcontroller/TMS_SWDIO -> /Microcontroller/PF5
- J4 pad 3: GND -> /Microcontroller/PF6
- J4 pad 4: /Microcontroller/TCK_SWDCLK -> /Microcontroller/PF7
- J4 pad 5: GND -> /Microcontroller/PF8
- J4 pad 6: /Microcontroller/TDO_SWO -> /Microcontroller/PF9
- J4 pad 7: Net-(J4-Pad7) -> /Microcontroller/PF10
- J4 pad 8: /Microcontroller/TDI -> /Microcontroller/PF11
- J4 pad 9: GND -> /Microcontroller/PF12
- R1 pad 2: Net-(R1-Pad2) -> VBUS
- R10 pad 1: /Level Shifter - I/O Pins 1&2/IO_1_OUT -> /Microcontroller/STATUS_R
- R10 pad 2: GND -> Net-(D3-Pad4)
- R11 pad 1: /Level Shifter - I/O Pins 1&2/~IO_1_TRIS -> /Microcontroller/STATUS_G
- R11 pad 2: Net-(D7-Pad1) -> Net-(D3-Pad2)
- R12 pad 1: /Level Shifter - I/O Pins 1&2/IO_2_OUT -> /Microcontroller/STATUS_B
- R12 pad 2: GND -> Net-(D3-Pad6)
- R2 pad 1: Net-(R2-Pad1) -> Net-(D1-Pad1)
- R2 pad 2: Net-(R2-Pad2) -> VBUS
- R3 pad 1: Net-(R3-Pad1) -> Net-(C11-Pad1)
- R3 pad 2: Net-(R3-Pad2) -> Net-(C12-Pad1)
- R4 pad 1: Net-(R4-Pad1) -> +3V3
- R4 pad 2: Net-(R4-Pad2) -> /Microcontroller/~INT_USBC
- R5 pad 1: Net-(D3-Pad1) -> Net-(R5-Pad1)
- R6 pad 1: Net-(D4-Pad1) -> Net-(D2-Pad1)
- R7 pad 1: Net-(D5-Pad2) -> Net-(R7-Pad1)
- R7 pad 2: GND -> Net-(R7-Pad2)
- R8 pad 1: Net-(D6-Pad1) -> +3V3
- R8 pad 2: GND -> /I2C_SCL
- R9 pad 1: /Microcontroller/OSC_OUT -> +3V3
- R9 pad 2: /Microcontroller/OSC_IN -> /I2C_SDA
- SW1 pad 2: Net-(R43-Pad2) -> Net-(R7-Pad2)
- SW1 pad 3: /3.3V -> +3V3
- SW2 pad 2: Net-(C28-Pad1) -> /Microcontroller/~RESET
- TP1 pad 1: Net-(R1-Pad1) -> GND
- TP2 pad 1: Net-(R1-Pad2) -> VBUS
- TP3 pad 1: Net-(Q1-Pad1) -> GND
- U1 pad 1: GND -> Net-(J1-PadA5)
- U1 pad 2: /3.3V -> Net-(J1-PadB5)
- U1 pad 3: /Vin -> GND
- U2 pad 1: Net-(TP51-Pad1) -> VBUS
- U2 pad 2: Net-(TP52-Pad1) -> GND
- U2 pad 3: Net-(TP53-Pad1) -> +3V3
- U2 pad 4: Net-(TP54-Pad1) -> (no net)
- U3 pad 10: Net-(U3-Pad10) -> (no net)
- U3 pad 14: /Microcontroller/ULPI_CK -> /Microcontroller/ULPI_CLK
- U3 pad 15: /Microcontroller/VDD1.8 -> /VDD1.8
- U3 pad 16: /3.3V -> +3V3
- U3 pad 25: /3.3V -> +3V3
- U3 pad 26: /Microcontroller/VDD1.8 -> /VDD1.8
- U3 pad 27: /Microcontroller/XO -> Net-(C11-Pad1)
- U3 pad 28: /Microcontroller/XI -> Net-(C12-Pad1)
- U3 pad 29: /Microcontroller/VDDA1.8 -> /VDDA1.8
- U3 pad 3: Net-(U3-Pad3) -> (no net)
- U3 pad 30: /3.3V -> +3V3
- U3 pad 31: /3.3V -> +3V3
- U3 pad 32: Net-(R45-Pad1) -> Net-(R5-Pad1)
- U3 pad 4: Net-(D12-Pad1) -> Net-(D1-Pad1)
- U3 pad 5: Net-(U3-Pad5) -> (no net)
- U3 pad 6: /3.3V -> +3V3
- U3 pad 7: /D+ -> /USB_D+
- U3 pad 8: /D- -> /USB_D-
- U3 pad 9: Net-(TP174-Pad1) -> /Microcontroller/ULPI_RESET
- U4 pad 1: GND -> /Microcontroller/PE2
- U4 pad 2: /3.3V -> /Microcontroller/PE3
- U4 pad 3: Net-(R47-Pad2) -> /Microcontroller/PE4
- U4 pad 4: Net-(C44-Pad2) -> /Microcontroller/PE5
- U4 pad 5: GND -> /Microcontroller/PE6
- U4 pad 6: /3.3V -> +3V3
- U4 pad 7: /Vin -> /Microcontroller/GPIO_PC13
- U4 pad 8: Net-(C43-Pad2) -> /Microcontroller/GPIO_PC14
- Y1 pad 1: /Microcontroller/OSC_OUT -> Net-(C11-Pad1)
- Y1 pad 3: /Microcontroller/OSC_IN -> Net-(C12-Pad1)
- Y2 pad 1: /Microcontroller/XO -> Net-(C33-Pad1)
- Y2 pad 3: /Microcontroller/XI -> Net-(C34-Pad1)
Routing:
- net CHASSIS: track 1019.9 -> 0.00 mm
- net /3.3V: track 957.8 -> 0.00 mm, vias 62 -> 0
- net /+15V: track 605.5 -> 0.00 mm, vias 40 -> 0
- net /-15V: track 541.8 -> 0.00 mm, vias 33 -> 0
- net GND: track 184.6 -> 0.00 mm, vias 293 -> 0
- net /Level Shifter - I/O Pins 1&2/I2C_SDA: track 169.6 -> 0.00 mm, vias 10 -> 0
- net /Level Shifter - I/O Pins 1&2/I2C_SCL: track 160.0 -> 0.00 mm, vias 12 -> 0
- net /Level Shifter - I/O Pins 3&4/IO_4_PU: track 140.0 -> 0.00 mm, vias 2 -> 0
- net /Level Shifter - I/O Pins 3&4/~IO_4_TRIS: track 121.2 -> 0.00 mm, vias 8 -> 0
- net /Level Shifter - I/O Pins 3&4/~IO_4_PD: track 119.7 -> 0.00 mm, vias 4 -> 0
- net /Level Shifter - I/O Pins 1&2/IO_2_OUT: track 119.2 -> 0.00 mm, vias 7 -> 0
- net /Level Shifter - I/O Pins 3&4/IO_4_OUT: track 118.6 -> 0.00 mm, vias 6 -> 0
- net /Level Shifter - I/O Pins 3&4/IO_3_OUT: track 117.9 -> 0.00 mm, vias 6 -> 0
- net /Level Shifter - I/O Pins 1&2/IO_1_OUT: track 117.1 -> 0.00 mm, vias 5 -> 0
- net /Vout: track 114.6 -> 0.00 mm, vias 2 -> 0
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- removed copper zone on F.Cu, net /+15V
- removed copper zone on F.Cu, net /-15V
- removed copper zone on F.Cu, net /3.3V
- removed copper zone on F.Cu, net /Vin
- removed copper zone on F.Cu, net /Vout
- removed copper zone on F.Cu, net CHASSIS
- removed copper zone on F.Cu, net GND
- removed copper zone on In1.Cu, net GND
- removed copper zone on In2.Cu, net GND
- removed copper zone on F.Cu, net Net-(C43-Pad1)
- removed copper zone on F.Cu, net Net-(C43-Pad2)
- removed copper zone on F.Cu, net Net-(D30-Pad2)
- removed copper zone on F.Cu, net Net-(D31-Pad1)
- removed copper zone on F.Cu, net Net-(L2-Pad1)
Other:
- board size 170 x 100 mm -> 75 x 110 mm
- copper layers 4 -> 2
- board text added: "2020-12-19"
- board text added: "I/O MASTER DEV BOARD v1.0"
- board text removed: "DC IN 5-12V"
- board text removed: "GND"
- board text removed: "I/O 1 OC"
- board text removed: "I/O 2 OC"
- board text removed: "I/O 3 OC"
- board text removed: "I/O 4 OC"
- board text removed: "IO1"
- board text removed: "IO2"
- board text removed: "IO3"
- board text removed: "IO4"
- board text removed: "VOUT"
