File: kicad/io-master-dev-board.sch (KiCad schematic (older format))
At the start: 46 parts, among them J1 USB4110-GF-A, J10 Conn_01x27, J2 Conn_01x08, J3 Conn_01x08, J4 Conn_01x12, J5 UART, J6 JUMPER, J7 JUMPER, J8 Conn_01x10, J9 Conn_01x32, U1 TUSB320, U2 K7803JT-500R3, U3 USB3300-EZK, Y1 24MHz

Commit message: WIP board layout
Parts:
- removed J6: JUMPER, Connector_PinHeader_2.54mm:PinHeader_2x32_P2.54mm_Vertical, symbol Connector_Generic:Conn_02x32_Counter_Clockwise
- removed J7: JUMPER, Connector_PinHeader_2.54mm:PinHeader_2x27_P2.54mm_Vertical, symbol Connector_Generic:Conn_02x27_Counter_Clockwise
- added J6: Conn_02x32_Odd_Even, Connector_PinHeader_1.27mm:PinHeader_2x32_P1.27mm_Vertical, symbol Connector_Generic:Conn_02x32_Odd_Even
- added J7: Conn_02x27_Odd_Even, Connector_PinHeader_1.27mm:PinHeader_2x27_P1.27mm_Vertical, symbol Connector_Generic:Conn_02x27_Odd_Even
- J10: footprint io-master-dev-board:Edge_PinHeader_1x27_P2.54mm_Horizontal -> Connector_PinHeader_1.27mm:PinHeader_1x27_P1.27mm_Vertical
- J8: footprint io-master-dev-board:Edge_PinHeader_1x10_P2.54mm_Horizontal -> Connector_PinHeader_1.27mm:PinHeader_1x10_P1.27mm_Vertical
- J9: footprint io-master-dev-board:Edge_PinHeader_1x32_P2.54mm_Horizontal -> Connector_PinHeader_1.27mm:PinHeader_1x32_P1.27mm_Vertical
Connections:
- net GND: now also H1.1, H2.1, H3.1, H4.1
- net Microcontroller/GPIO_PA11: now also J7.5 (Pin_5)
- net Microcontroller/GPIO_PA12: now also J7.7 (Pin_7)
- net Microcontroller/GPIO_PA4: now also J7.1 (Pin_1)
- net Microcontroller/GPIO_PA6: now also J7.3 (Pin_3)
- net Microcontroller/GPIO_PB14: now also J7.13 (Pin_13)
- net Microcontroller/GPIO_PB15: now also J7.15 (Pin_15)
- net Microcontroller/GPIO_PB2: now also J7.9 (Pin_9)
- net Microcontroller/GPIO_PB6: now also J7.11 (Pin_11)
- net Microcontroller/GPIO_PC1: now also J7.17 (Pin_17)
- net Microcontroller/GPIO_PC10: now also J7.27 (Pin_27)
- net Microcontroller/GPIO_PC11: now also J7.29 (Pin_29)
- net Microcontroller/GPIO_PC12: now also J7.31 (Pin_31)
- net Microcontroller/GPIO_PC13: now also J7.33 (Pin_33)
- net Microcontroller/GPIO_PC14: now also J7.35 (Pin_35)
- net Microcontroller/GPIO_PC15: now also J7.37 (Pin_37)
- net Microcontroller/GPIO_PC4: now also J7.19 (Pin_19)
- net Microcontroller/GPIO_PC5: now also J7.21 (Pin_21)
- net Microcontroller/GPIO_PC7: now also J7.23 (Pin_23)
- net Microcontroller/GPIO_PC8: now also J7.25 (Pin_25)
- net Microcontroller/GPIO_PG0: now also J7.39 (Pin_39)
- net Microcontroller/GPIO_PG1: now also J7.41 (Pin_41)
- net Microcontroller/GPIO_PG2: now also J7.43 (Pin_43)
- net Microcontroller/GPIO_PG3: now also J7.45 (Pin_45)
- net Microcontroller/GPIO_PG4: now also J7.47 (Pin_47)
- net Microcontroller/GPIO_PG5: now also J7.49 (Pin_49)
- net Microcontroller/GPIO_PG6: now also J7.51 (Pin_51)
- net Microcontroller/GPIO_PG7: now also J7.53 (Pin_53)
- net Microcontroller/IO_1_CLK: now also J6.3 (Pin_3)
- net Microcontroller/IO_1_IN: now also J6.7 (Pin_7)
- net Microcontroller/IO_1_OUT: now also J6.1 (Pin_1)
- net Microcontroller/IO_2_CLK: now also J6.11 (Pin_11)
- net Microcontroller/IO_2_IN: now also J6.15 (Pin_15)
- net Microcontroller/IO_2_OUT: now also J6.9 (Pin_9)
- net Microcontroller/IO_3_CLK: now also J6.19 (Pin_19)
- net Microcontroller/IO_3_IN: now also J6.23 (Pin_23)
- net Microcontroller/IO_3_OUT: now also J6.17 (Pin_17)
- net Microcontroller/IO_4_CLK: now also J6.27 (Pin_27)
- net Microcontroller/IO_4_IN: now also J6.31 (Pin_31)
- net Microcontroller/IO_4_OUT: now also J6.25 (Pin_25)
- net Microcontroller/IO_5_CLK: now also J6.35 (Pin_35)
- net Microcontroller/IO_5_IN: now also J6.39 (Pin_39)
- net Microcontroller/IO_5_OUT: now also J6.33 (Pin_33)
- net Microcontroller/IO_6_CLK: now also J6.43 (Pin_43)
- net Microcontroller/IO_6_IN: now also J6.47 (Pin_47)
- net Microcontroller/IO_6_OUT: now also J6.41 (Pin_41)
- net Microcontroller/IO_7_CLK: now also J6.51 (Pin_51)
- net Microcontroller/IO_7_IN: now also J6.55 (Pin_55)
- net Microcontroller/IO_7_OUT: now also J6.49 (Pin_49)
- net Microcontroller/IO_8_CLK: now also J6.59 (Pin_59)
- net Microcontroller/IO_8_IN: now also J6.63 (Pin_63)
- net Microcontroller/IO_8_OUT: now also J6.57 (Pin_57)
- net Microcontroller/~IO_1_TRIS: now also J6.5 (Pin_5)
- net Microcontroller/~IO_2_TRIS: now also J6.13 (Pin_13)
- net Microcontroller/~IO_3_TRIS: now also J6.21 (Pin_21)
- net Microcontroller/~IO_4_TRIS: now also J6.29 (Pin_29)
- net Microcontroller/~IO_5_TRIS: now also J6.37 (Pin_37)
- net Microcontroller/~IO_6_TRIS: now also J6.45 (Pin_45)
- net Microcontroller/~IO_7_TRIS: now also J6.53 (Pin_53)
- net Microcontroller/~IO_8_TRIS: now also J6.61 (Pin_61)
- net at J9.1 (Pin_1): now also J6.2 (Pin_2)
- net at J9.10 (Pin_10): now also J6.20 (Pin_20)
- net at J9.11 (Pin_11): now also J6.22 (Pin_22)
- net at J9.12 (Pin_12): now also J6.24 (Pin_24)
- net at J9.13 (Pin_13): now also J6.26 (Pin_26)
- net at J9.14 (Pin_14): now also J6.28 (Pin_28)
- net at J9.15 (Pin_15): now also J6.30 (Pin_30)
- net at J9.16 (Pin_16): now also J6.32 (Pin_32)
- net at J9.17 (Pin_17): now also J6.34 (Pin_34)
- net at J9.18 (Pin_18): now also J6.36 (Pin_36)
- net at J9.19 (Pin_19): now also J6.38 (Pin_38)
- net at J9.2 (Pin_2): now also J6.4 (Pin_4)
- net at J9.20 (Pin_20): now also J6.40 (Pin_40)
- net at J9.21 (Pin_21): now also J6.42 (Pin_42)
- net at J9.22 (Pin_22): now also J6.44 (Pin_44)
- net at J9.23 (Pin_23): now also J6.46 (Pin_46)
- net at J9.24 (Pin_24): now also J6.48 (Pin_48)
- net at J9.25 (Pin_25): now also J6.50 (Pin_50)
- net at J9.26 (Pin_26): now also J6.52 (Pin_52)
- net at J9.27 (Pin_27): now also J6.54 (Pin_54)
- net at J9.28 (Pin_28): now also J6.56 (Pin_56)
- net at J9.29 (Pin_29): now also J6.58 (Pin_58)
- net at J9.3 (Pin_3): now also J6.6 (Pin_6)
- net at J9.30 (Pin_30): now also J6.60 (Pin_60)
- net at J9.31 (Pin_31): now also J6.62 (Pin_62)
- net at J9.32 (Pin_32): now also J6.64 (Pin_64)
- net at J9.4 (Pin_4): now also J6.8 (Pin_8)
- net at J9.5 (Pin_5): now also J6.10 (Pin_10)
- net at J9.6 (Pin_6): now also J6.12 (Pin_12)
- net at J9.7 (Pin_7): now also J6.14 (Pin_14)
- net at J9.8 (Pin_8): now also J6.16 (Pin_16)
- net at J9.9 (Pin_9): now also J6.18 (Pin_18)
- net at J10.1 (Pin_1): now also J7.2 (Pin_2)
- net at J10.10 (Pin_10): now also J7.20 (Pin_20)
- net at J10.11 (Pin_11): now also J7.22 (Pin_22)
- net at J10.12 (Pin_12): now also J7.24 (Pin_24)
- net at J10.13 (Pin_13): now also J7.26 (Pin_26)
- net at J10.14 (Pin_14): now also J7.28 (Pin_28)
- net at J10.15 (Pin_15): now also J7.30 (Pin_30)
- net at J10.16 (Pin_16): now also J7.32 (Pin_32)
- net at J10.17 (Pin_17): now also J7.34 (Pin_34)
- net at J10.18 (Pin_18): now also J7.36 (Pin_36)
- net at J10.19 (Pin_19): now also J7.38 (Pin_38)
- net at J10.2 (Pin_2): now also J7.4 (Pin_4)
- net at J10.20 (Pin_20): now also J7.40 (Pin_40)
- net at J10.21 (Pin_21): now also J7.42 (Pin_42)
- net at J10.22 (Pin_22): now also J7.44 (Pin_44)
- net at J10.23 (Pin_23): now also J7.46 (Pin_46)
- net at J10.24 (Pin_24): now also J7.48 (Pin_48)
- net at J10.25 (Pin_25): now also J7.50 (Pin_50)
- net at J10.26 (Pin_26): now also J7.52 (Pin_52)
- net at J10.27 (Pin_27): now also J7.54 (Pin_54)
- net at J10.3 (Pin_3): now also J7.6 (Pin_6)
- net at J10.4 (Pin_4): now also J7.8 (Pin_8)
- net at J10.5 (Pin_5): now also J7.10 (Pin_10)
- net at J10.6 (Pin_6): now also J7.12 (Pin_12)
- net at J10.7 (Pin_7): now also J7.14 (Pin_14)
- net at J10.8 (Pin_8): now also J7.16 (Pin_16)
- net at J10.9 (Pin_9): now also J7.18 (Pin_18)
- removed net CHASSIS: C7.2, H1.1, H2.1, H3.1, H4.1, J1.S1 (SHIELD)
- new net: C7.2, J1.S1 (SHIELD)
Other:
- note added: "NOTE: DECOUPLING CAPS FOR U3 VDD3.3 PINS"
- note added: "NOTE: DECOUPLING CAPS\nFOR U3 VDD1.8 PINS"
- note added: "NOTE: DECOUPLING CAPS\nFOR U3 VDDA1.8 PIN"
- note added: "NOTE: DECOUPLING CAP\nFOR U1 VDD PIN"
- note removed: "NOTE: DECOUPLING CAPS FOR U? VDD3.3 PINS"
- note removed: "NOTE: DECOUPLING CAPS\nFOR U? VDD1.8 PINS"
- note removed: "NOTE: DECOUPLING CAPS\nFOR U? VDDA1.8 PIN"
- note removed: "NOTE: DECOUPLING CAP\nFOR U? VDD PIN"
- moved on the sheet: C7
Changed lines of the file:
@@
 L power:GND #PWR06
 U 1 1 5FD5664C
-P 2450 3450
-F 0 "#PWR06" H 2450 3200 50  0001 C CNN
-F 1 "GND" H 2455 3277 50  0000 C CNN
-F 2 "" H 2450 3450 50  0001 C CNN
-F 3 "" H 2450 3450 50  0001 C CNN
-	1    2450 3450
-	1    0    0    -1
-$EndComp
-Wire Wire Line
-	1950 3050 1950 3250
-Wire Wire Line
-	2450 3100 2450 3250
-Connection ~ 1950 3250
-Wire Wire Line
-	1950 3250 1950 3450
-Connection ~ 2450 3250
-Wire Wire Line
-	2450 3250 2450 3450
-Wire Wire Line
-	1950 3250 2050 3250
-Wire Wire Line
-	2350 3250 2450 3250
+P 1950 3500
+F 0 "#PWR06" H 1950 3250 50  0001 C CNN
+F 1 "GND" H 1955 3327 50  0000 C CNN
+F 2 "" H 1950 3500 50  0001 C CNN
+F 3 "" H 1950 3500 50  0001 C CNN
+	1    1950 3500
+	1    0    0    -1
+$EndComp
 $Comp
 L Device:C C7
 U 1 1 5FD5666A
-P 2200 3250
-F 0 "C7" V 2050 3100 50  0000 L CNN
-F 1 "0.1u" V 2050 3250 50  0000 L CNN
-F 2 "Capacitor_SMD:C_0603_1608Metric" H 2238 3100 50  0001 C CNN
-F 3 "~" H 2200 3250 50  0001 C CNN
-	1    2200 3250
-	0    1    -1   0
+P 1950 3250
+F 0 "C7" H 2050 3200 50  0000 L CNN
+F 1 "0.1u" H 2050 3300 50  0000 L CNN
+F 2 "Capacitor_SMD:C_0603_1608Metric" H 1988 3100 50  0001 C CNN
+F 3 "~" H 1950 3250 50  0001 C CNN
+	1    1950 3250
+	-1   0    0    1
 $EndComp
 Wire Wire Line
@@
 	6100 7450 6100 7500
 Text Notes 950  7200 0    50   ~ 0
-NOTE: DECOUPLING CAPS\nFOR U? VDD1.8 PINS
+NOTE: DECOUPLING CAPS\nFOR U3 VDD1.8 PINS
 $Comp
 L power:GND #PWR024
@@
 	1450 6600 1900 6600
 Text Notes 950  5900 0    50   ~ 0
-NOTE: DECOUPLING CAPS FOR U? VDD3.3 PINS
+NOTE: DECOUPLING CAPS FOR U3 VDD3.3 PINS
 NoConn ~ 6150 6950
 NoConn ~ 6150 6350
@@
 	3200 7350 3200 7400
 Text Notes 2550 7200 0    50   ~ 0
-NOTE: DECOUPLING CAPS\nFOR U? VDDA1.8 PIN
+NOTE: DECOUPLING CAPS\nFOR U3 VDDA1.8 PIN
 $Comp
 L Device:R R3
@@
 	-1   0    0    -1
 $EndComp
-Wire Wire Line
-	2250 3050 2250 3100
-Wire Wire Line
-	2250 3100 2450 3100
 $Comp
 L power:VBUS #PWR09
@@
 I2C ADDRESS SELECTION:\n  HIGH JUMPER: 0x61\n  LOW JUMPER: 0x60 (DEFAULT)\n
 Text Notes 7050 2400 0    50   ~ 0
-NOTE: DECOUPLING CAP\nFOR U? VDD PIN
+NOTE: DECOUPLING CAP\nFOR U1 VDD PIN
 Wire Wire Line
 	1000 9650 1000 9600
@@
 STM32H7\nMICROCONTROLLER
 $Comp
-L io-master-dev-board:CHASSIS #PWR05
-U 1 1 6166FC9A
-P 1950 3450
-F 0 "#PWR05" H 1950 3250 50  0001 C CNN
-F 1 "CHASSIS" H 1954 3296 50  0000 C CNN
-F 2 "" H 1950 3400 50  0001 C CNN
-F 3 "" H 1950 3400 50  0001 C CNN
-	1    1950 3450
-	1    0    0    -1
-$EndComp
-$Comp
-L io-master-dev-board:CHASSIS #PWR04
-U 1 1 616708D0
-P 1000 9700
-F 0 "#PWR04" H 1000 9500 50  0001 C CNN
-F 1 "CHASSIS" H 1004 9546 50  0000 C CNN
-F 2 "" H 1000 9650 50  0001 C CNN
-F 3 "" H 1000 9650 50  0001 C CNN
-	1    1000 9700
-	1    0    0    -1
-$EndComp
-$Comp
 L Connector_Generic:Conn_01x10 J8
 U 1 1 616874B9
@@
 F 0 "J8" H 14600 1950 50  0000 C CNN
 F 1 "Conn_01x10" H 14680 1351 50  0001 L CNN
-F 2 "io-master-dev-board:Edge_PinHeader_1x10_P2.54mm_Horizontal" H 14600 1450 50  0001 C CNN
+F 2 "Connector_PinHeader_1.27mm:PinHeader_1x10_P1.27mm_Vertical" H 14600 1450 50  0001 C CNN
 F 3 "~" H 14600 1450 50  0001 C CNN
 	1    14600 1450
@@
 F 0 "J9" H 14600 5450 50  0000 C CNN
 F 1 "Conn_01x32" H 14680 3751 50  0001 L CNN
-F 2 "io-master-dev-board:Edge_PinHeader_1x32_P2.54mm_Horizontal" H 14600 3850 50  0001 C CNN
+F 2 "Connector_PinHeader_1.27mm:PinHeader_1x32_P1.27mm_Vertical" H 14600 3850 50  0001 C CNN
 F 3 "~" H 14600 3850 50  0001 C CNN
 	1    14600 3850
@@
 F 0 "J10" H 14600 8550 50  0000 C CNN
 F 1 "Conn_01x27" H 14680 7101 50  0001 L CNN
-F 2 "io-master-dev-board:Edge_PinHeader_1x27_P2.54mm_Horizontal" H 14600 7150 50  0001 C CNN
+F 2 "Connector_PinHeader_1.27mm:PinHeader_1x27_P1.27mm_Vertical" H 14600 7150 50  0001 C CNN
 F 3 "~" H 14600 7150 50  0001 C CNN
 	1    14600 7150
@@
 Wire Wire Line
 	13550 5850 13750 5850
-$Comp
-L Connector_Generic:Conn_02x32_Counter_Clockwise J6
-U 1 1 608EF63F
-P 13950 3850
-F 0 "J6" H 14000 5450 50  0000 C CNN
-F 1 "JUMPER" H 14000 2150 50  0000 C CNN
-F 2 "Connector_PinHeader_2.54mm:PinHeader_2x32_P2.54mm_Vertical" H 13950 3850 50  0001 C CNN
-F 3 "~" H 13950 3850 50  0001 C CNN
-	1    13950 3850
-	1    0    0    -1
-$EndComp
 Wire Wire Line
 	14250 2350 14400 2350
@@
 Wire Wire Line
 	13750 2850 13550 2850
-$Comp
-L Connector_Generic:Conn_02x27_Counter_Clockwise J7
-U 1 1 608FFD5B
-P 13950 7150
-F 0 "J7" H 14000 8550 50  0000 C CNN
-F 1 "JUMPER" H 14000 5750 50  0000 C CNN
-F 2 "Connector_PinHeader_2.54mm:PinHeader_2x27_P2.54mm_Vertical" H 13950 7150 50  0001 C CNN
-F 3 "~" H 13950 7150 50  0001 C CNN
-	1    13950 7150
-	1    0    0    -1
-$EndComp
 Wire Wire Line
 	14250 5850 14400 5850
@@
 Text Label 13650 1750 0    50   ~ 0
 I2C_SCL
+$Comp
+L power:GND #PWR0101
+U 1 1 5FD88D31
+P 1000 9700
+F 0 "#PWR0101" H 1000 9450 50  0001 C CNN
+F 1 "GND" H 1005 9527 50  0000 C CNN
+F 2 "" H 1000 9700 50  0001 C CNN
+F 3 "" H 1000 9700 50  0001 C CNN
+	1    1000 9700
+	1    0    0    -1
+$EndComp
+Wire Wire Line
+	1950 3050 1950 3100
+Wire Wire Line
+	1950 3500 1950 3450
+Wire Wire Line
+	2250 3450 1950 3450
+Connection ~ 1950 3450
+Wire Wire Line
+	1950 3450 1950 3400
+Wire Wire Line
+	2250 3050 2250 3450
+$Comp
+L Connector_Generic:Conn_02x32_Odd_Even J6
+U 1 1 5FE52FA7
+P 13950 3850
+F 0 "J6" H 14000 5450 50  0000 C CNN
+F 1 "Conn_02x32_Odd_Even" H 14000 5476 50  0001 C CNN
+F 2 "Connector_PinHeader_1.27mm:PinHeader_2x32_P1.27mm_Vertical" H 13950 3850 50  0001 C CNN
+F 3 "~" H 13950 3850 50  0001 C CNN
+	1    13950 3850
+	1    0    0    -1
+$EndComp
+$Comp
+L Connector_Generic:Conn_02x27_Odd_Even J7
+U 1 1 5FE5FFF1
+P 13950 7150
+F 0 "J7" H 14000 8550 50  0000 C CNN
+F 1 "Conn_02x27_Odd_Even" H 14000 8576 50  0001 C CNN
+F 2 "Connector_PinHeader_1.27mm:PinHeader_2x27_P1.27mm_Vertical" H 13950 7150 50  0001 C CNN
+F 3 "~" H 13950 7150 50  0001 C CNN
+	1    13950 7150
+	1    0    0    -1
+$EndComp
 $EndSCHEMATC
